File: schematic/master_mcu.kicad_sch (KiCad schematic)
At the start: 11 parts, among them U1 HC-SR04, U10 TCRT5000, U2 HC-SR04, U3 HC-SR04, U5 LSM9DS1, U6 HC-SR04, U7 TCRT5000, U8 TCRT5000, U9 TCRT5000

Commit message: updated schematic
Parts:
- removed U10, U9: TCRT5000, symbol symbol_lib:TCRT5000
- removed U3, U6: HC-SR04, symbol symbol_lib:HC-SR04
- removed U5: LSM9DS1, Package_LGA:LGA-24L_3x3.5mm_P0.43mm, symbol Sensor_Motion:LSM9DS1
- added C2, C3: 0.1uF, symbol Device:C
- added C4, C5: 47nF, symbol Device:C
- added Q1, Q2: LTR-3208E, symbol Device:Q_Photo_NPN_CE
- added R1, R19, R2, R20, R3, R4, R7, R8: 10K, symbol Device:R
- added R10, R13, R14, R15, R16, R17, R18, R5, R6, R9: 1K, symbol Device:R
- added R11, R12: 240K, symbol Device:R
- added R21, R22: 4.7K, symbol Device:R
- added U10, U11: LM339, symbol Comparator:LM339
- added U6, U7, U8, U9: MCP6294, Package_TO_SOT_SMD:SOT-23-5, symbol Amplifier_Operational:MCP6001-OT
- renumbered A2 to A1, U1 to U2, U7 to U3, U2 to U4, U8 to U5
Connections:
- net +5V: now also C2.1, C3.1, Q1.1 (C), Q2.1 (C), R1.1, R13.1, R14.1, R17.1, R18.1, R21.1, R22.1, R3.1, U6.5 (V+), U7.5 (V+), U8.5 (V+), U9.5 (V+)
- net GND: now also C2.2, C3.2, R10.2, R15.2, R16.2, R2.2, R4.2, R5.2, R6.2, R9.2, U6.2 (V-), U7.2 (V-), U8.2 (V-), U9.2 (V-)
- net A2_M: no longer names the net of A1.11 (A2)
- net A3_M: no longer names the net of A1.12 (A3)
- net D12_M: no longer names the net of A1.27 (D12)
- net D8_M: no longer names the net of A1.23 (D8)
- new net: R3.2, R4.1, U7.3 (+)
- new net: C5.1, Q2.2 (E), R6.1
- new net: C4.2, R7.1, U8.3 (+)
- new net: R11.2, U10.4 (-), U8.1
- new net: R11.1, R9.1, U8.4 (-)
- new net: R1.2, R2.1, U6.3 (+)
- new net: R12.2, U11.4 (-), U9.1
- new net: C5.2, R8.1, U9.3 (+)
- new net: R10.1, R12.1, U9.4 (-)
- new net: R14.2, R16.1, R18.2, R20.1, U11.5 (+)
- new net: R20.2, R22.2, U11.2
- new net: R13.2, R15.1, R17.2, R19.1, U10.5 (+)
- new net: C4.1, Q1.2 (E), R5.1
- new net: R19.2, R21.2, U10.2
- new net Vref1: R7.2, R8.2, U6.1, U6.4 (-)
- new net Vref2: U7.1, U7.4 (-)
- no-connect marks 34 -> 20
Other:
- note added: "At the comparator"
- note added: "At the op-amp"
- note added: "Cutoff Frequency: ~338Hz. Highest frequency to detect: 3.3kHz Lowest frequency to detect: 900Hz"
- note added: "IR Receivers"
- note added: "Nominal gain: ~240x"
- note added: "Theoretical hysteresis boundaries (disregarding 4.7k pullup): 3.23V and 3.34V"
- note added: "Unity Gain Buffers"
- note removed: "LSM9DS1 9-DOF Sensor"
- note removed: "Will look into specifics later"
- moved on the sheet: A1, C1, U2, U3, U4, U5
