File: schematic/core_mcu.kicad_sch (KiCad schematic)
At the start: 40 parts, among them Q1 LTR-3208E, Q2 LTR-3208E, U10 LM339, U11 LM339, U2 HC-SR04, U3 TCRT5000, U4 HC-SR04, U5 TCRT5000, U6 MCP6294, U7 MCP6294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

Commit message: update schematics
Parts:
- added U14, U15: TCRT5000, symbol symbol_lib:TCRT5000
Connections:
- net D2_M is gone; now on net D2_C: A1.17 (D2)
- net D9_M is gone; now on net D9_C: U2.2 (Trig), U4.2 (Trig)
- net +5V: now also U14.1 (VCC), U15.1 (VCC)
- net GND: now also U14.2 (GND), U15.2 (GND)
- net D2_C: now reaches R20.2, R22.2, U11.2
- net A2_C: now reaches A1.11 (A2)
- net A2_C: now also U14.4 (A0)
- net A3_C: now reaches A1.12 (A3)
- net A3_C: now also U15.4 (A0)
- net D3_C: now reaches A1.18 (D3)
- net D3_C: now also R19.2, R21.2, U10.2
- net D9_C: now reaches A1.24 (D9)
- net A0_M renamed A0_C
- net A1_M renamed A1_C
- net D4_M renamed D4_C
- net D7_M renamed D7_C
- no-connect marks 20 -> 18
Other:
- moved on the sheet: A1

Commit message: updated schematic
Connections:
- net GND: no longer R10.2, R9.2
- net Vref1: now also R10.2; no longer R7.2
- net Vref2: now also R7.2, R9.2
Changed lines of the file:
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@@
 	(wire
 		(pts
+			(xy 195.58 63.5) (xy 195.58 78.74)
+		)
+		(stroke
+			(width 0)
+			(type default)
+		)
+	)
+	(wire
+		(pts
 			(xy 50.8 68.58) (xy 43.18 68.58)
 		)
@@
 	(wire
 		(pts
-			(xy 195.58 63.5) (xy 195.58 69.85)
-		)
-		(stroke
-			(width 0)
-			(type default)
-		)
-	)
-	(wire
-		(pts
 			(xy 173.99 49.53) (xy 173.99 53.34)
 		)
@@
 	(wire
 		(pts
+			(xy 194.31 135.89) (xy 194.31 148.59)
+		)
+		(stroke
+			(width 0)
+			(type default)
+		)
+	)
+	(wire
+		(pts
 			(xy 29.21 149.86) (xy 36.83 149.86)
 		)
@@
 	(wire
 		(pts
-			(xy 194.31 116.84) (xy 194.31 128.27)
-		)
-		(stroke
-			(width 0)
-			(type default)
-		)
-	)
-	(wire
-		(pts
 			(xy 73.66 35.56) (xy 67.31 35.56)
 		)
@@
 	(wire
 		(pts
-			(xy 194.31 135.89) (xy 194.31 142.24)
+			(xy 133.35 26.67) (xy 133.35 31.75)
 		)
 		(stroke
@@
 	(wire
 		(pts
-			(xy 133.35 26.67) (xy 133.35 31.75)
+			(xy 50.8 86.36) (xy 43.18 86.36)
 		)
 		(stroke
@@
 	(wire
 		(pts
-			(xy 50.8 86.36) (xy 43.18 86.36)
+			(xy 233.68 43.18) (xy 237.49 43.18)
 		)
 		(stroke
@@
 	(wire
 		(pts
-			(xy 233.68 43.18) (xy 237.49 43.18)
+			(xy 264.16 31.75) (xy 264.16 35.56)
 		)
 		(stroke
@@
 	(wire
 		(pts
-			(xy 264.16 31.75) (xy 264.16 35.56)
+			(xy 233.68 35.56) (xy 237.49 35.56)
 		)
 		(stroke
@@
 	(wire
 		(pts
-			(xy 233.68 35.56) (xy 237.49 35.56)
+			(xy 194.31 116.84) (xy 194.31 128.27)
 		)
 		(stroke
@@
 		)
 	)
+	(label "Vref1"
+		(at 195.58 73.66 90)
+		(fields_autoplaced yes)
+		(effects
+			(font
+				(size 1.27 1.27)
+			)
+			(justify left bottom)
+		)
+	)
 	(label "D2_C"
 		(at 266.7 49.53 0)
@@
 		)
 	)
+	(label "Vref2"
+		(at 194.31 143.51 90)
+		(fields_autoplaced yes)
+		(effects
+			(font
+				(size 1.27 1.27)
+			)
+			(justify left bottom)
+		)
+	)
 	(label "+5V"
 		(at 48.26 66.04 180)
@@
 		)
 	)
-	(label "Vref1"
+	(label "Vref2"
 		(at 172.72 143.51 90)
 		(fields_autoplaced yes)
@@
 	)
 	(symbol
-		(lib_id "power:GND")
-		(at 195.58 69.85 0)
-		(unit 1)
-		(exclude_from_sim no)
-		(in_bom yes)
-		(on_board yes)
-		(dnp no)
-		(fields_autoplaced yes)
-		(property "Reference" "#PWR029"
-			(at 195.58 76.2 0)
-			(effects
-				(font
-					(size 1.27 1.27)
-				)
-				(hide yes)
-			)
-		)
-		(property "Value" "GND"
-			(at 195.58 74.93 0)
-			(effects
-				(font
-					(size 1.27 1.27)
-				)
-			)
-		)
-		(property "Footprint" ""
-			(at 195.58 69.85 0)
-			(effects
-				(font
-					(size 1.27 1.27)
-				)
-				(hide yes)
-			)
-		)
-		(property "Datasheet" ""
-			(at 195.58 69.85 0)
-			(effects
-				(font
-					(size 1.27 1.27)
-				)
-				(hide yes)
-			)
-		)
-		(property "Description" "Power symbol creates a global label with name \"GND\" , ground"
-			(at 195.58 69.85 0)
-			(effects
-				(font
-					(size 1.27 1.27)
-				)
-				(hide yes)
-			)
-		)
-		(pin "1"
-		)
-		(instances
-			(project "schematic"
-				(path "/a117cae9-da48-465a-8dd5-c903415f43a6/36720b7f-9e6e-4197-8c28-207631d2c0a5"
-					(reference "#PWR029")
-					(unit 1)
-				)
-			)
-		)
-	)
-	(symbol
 		(lib_id "power:+5V")
 		(at 154.94 29.21 0)
@@
 					(unit 1)
 				)
-			)
-		)
-	)
-	(symbol
-		(lib_id "power:GND")
-		(at 194.31 142.24 0)
-		(unit 1)
-		(exclude_from_sim no)
-		(in_bom yes)
-		(on_board yes)
-		(dnp no)
-		(fields_autoplaced yes)
-		(property "Reference" "#PWR028"
-			(at 194.31 148.59 0)
-			(effects
-				(font
-					(size 1.27 1.27)
-				)
-				(hide yes)
-			)
-		)
-		(property "Value" "GND"
-			(at 194.31 147.32 0)
-			(effects
-				(font
-					(size 1.27 1.27)
-				)
-			)
-		)
-		(property "Footprint" ""
-			(at 194.31 142.24 0)
-			(effects
-				(font
-					(size 1.27 1.27)
-				)
-				(hide yes)
-			)
-		)
-		(property "Datasheet" ""
-			(at 194.31 142.24 0)
-			(effects
-				(font
-					(size 1.27 1.27)
-				)
-				(hide yes)
-			)
-		)
-		(property "Description" "Power symbol creates a global label with name \"GND\" , ground"
-			(at 194.31 142.24 0)
-			(effects
-				(font
-					(size 1.27 1.27)
-				)
-				(hide yes)
-			)
-		)
-		(pin "1"
-		)
-		(instances
-			(project "schematic"
-				(path "/a117cae9-da48-465a-8dd5-c903415f43a6/36720b7f-9e6e-4197-8c28-207631d2c0a5"
-					(reference "#PWR028")
-					(unit 1)
-				)

Commit message: update schematic to match most recent config
Parts:
- removed C1: 100uF, symbol Device:C
- removed C2, C3: 0.1uF, symbol Device:C
- removed C4, C5: 47nF, symbol Device:C
- removed Q1, Q2: LTR-3208E, symbol Device:Q_Photo_NPN_CE
- removed R1, R19, R2, R20, R3, R4, R7, R8: 10K, symbol Device:R
- removed R10, R13, R14, R15, R16, R17, R18, R5, R6, R9: 1K, symbol Device:R
- removed R11, R12: 240K, symbol Device:R
- removed R21, R22: 4.7K, symbol Device:R
- removed U10, U11: LM339, symbol Comparator:LM339
- removed U6, U7, U8, U9: MCP6294, Package_TO_SOT_SMD:SOT-23-5, symbol Amplifier_Operational:MCP6001-OT
Connections:
- net D9_C: no longer U2.2 (Trig)
- net D10_C: now reaches A1.25 (D10)
- net D10_C: now also U2.2 (Trig)
- net D2_C: no longer names the net of A1.17 (D2)
- net D3_C: no longer names the net of A1.18 (D3)
- no-connect marks 18 -> 19
Other:
- note removed: "At the comparator"
- note removed: "At the op-amp"
- note removed: "At the power rail"
- note removed: "Cutoff Frequency: ~338Hz. Highest frequency to detect: 3.3kHz Lowest frequency to detect: 900Hz"
- note removed: "IR Receivers"
- note removed: "Nominal gain: ~240x"
- note removed: "Theoretical hysteresis boundaries (disregarding 4.7k pullup): 3.23V and 3.34V"
- note removed: "Unity Gain Buffers"
- moved on the sheet: A1, U14, U15, U2, U3, U4, U5
